Commit message: Setup mountain in simulation run_creature method

File: test.urdf (robot description, URDF)
Before this commit: robot pepe, 5 links, 4 joints
Links:
- removed link 24
- link 0: mass 2.566253749236391 -> 0.8691109574392354; geometry collision cylinder length=0.7925274666538502 radius=0.5908204445669372; visual cylinder length=0.7925274666538502 radius=0.5908204445669372
- link 11: mass 0.5872104307915559 -> 1.2043052937645218; geometry collision cylinder length=1.748595271566875 radius=0.4682186533095304; visual cylinder length=1.748595271566875 radius=0.4682186533095304
- link 22: mass 0.792167904531086 -> 1.9914942514486305; geometry collision cylinder length=0.6452539002315998 radius=0.9911725661694395; visual cylinder length=0.6452539002315998 radius=0.9911725661694395
- link 23: mass 0.792167904531086 -> 1.9914942514486305; geometry collision cylinder length=0.6452539002315998 radius=0.9911725661694395; visual cylinder length=0.6452539002315998 radius=0.9911725661694395
Joints:
- removed joint 24_to_11
- joint 11_to_0: axis 1 0 0 -> 0 0 1; origin xyz=0.6460731409149567 0.5892215424856213 0.3378550388942536 rpy=8.022872907415868 1.3987671371920307 3.558036816189643 -> xyz=0.32167119751525974 0.9901643167309767 0.8239329535751035 rpy=3.999815934606585 4.7315075324993865 0.7199631731704103
- joint 22_to_11: axis 0 1 0 -> 0 0 1; origin xyz=0.31742304581361014 0.9780298507842675 0.29975081908846724 rpy=9.46460064565625 3.338614172679243 0.49146827478779825 -> xyz=0.5691185762797627 0.47116934899365337 0.9157616669417802 rpy=1.6376076543688558 0.7409839306171004 3.5804341756472415
- joint 23_to_11: axis 0 1 0 -> 0 0 1; origin xyz=0.31742304581361014 0.9780298507842675 0.29975081908846724 rpy=14.196900968484375 3.338614172679243 0.49146827478779825 -> xyz=0.5691185762797627 0.47116934899365337 0.9157616669417802 rpy=2.4564114815532836 0.7409839306171004 3.5804341756472415
